File: Hardware/Kicad/ProjetSemestreKicad.kicad_pcb (KiCad board)
At the start: 2 copper layers, 5 parts, among them U1 DS18B20

Commit message: Kicadupdated
Parts:
- added R2: 1K, Resistor_THT:R_Axial_DIN0207_L6.3mm_D2.5mm_P7.62mm_Horizontal, F.Cu at (71.1, 66.0)
- added R3: 1K, Resistor_THT:R_Axial_DIN0207_L6.3mm_D2.5mm_P7.62mm_Horizontal, F.Cu at (71.1, 61.0)
- added SOL+1: MountingHole_Pad, Connector_Pin:Pin_D1.0mm_L10.0mm, F.Cu at (78.7, 71.1)
- added SOL-1: MountingHole_Pad, Connector_Pin:Pin_D1.0mm_L10.0mm, F.Cu at (73.7, 71.1)
- moved GND1 15.2 mm to (71.1, 38.1)
- moved DCIN1 11.4 mm to (71.1, 33.0)
- moved R1 5.08 mm to (71.1, 49.5)
- moved U1 5.08 mm to (78.7, 52.1)
Connections:
- A1 pad 20: unconnected-(A1-A1-Pad20) -> Net-(A1-A1)
Routing:
- net GND: track 47.8 -> 63.8 mm
- net Net-(A1-A1): track 0.00 -> 15.6 mm
- net Net-(R2-Pad2): track 0.00 -> 5.08 mm
- net Net-(A1-A0): track 20.9 -> 15.9 mm
- net Net-(A1-+5V): track 23.3 -> 21.2 mm
- net Net-(A1-VIN): track 7.62 -> 6.13 mm
- added copper zone on B.Cu, net GND
Other:
- board outline added: 17.8 x 45.7 mm
