File: Hardware/Kicad/ProjetSemestreKicad.kicad_sch (KiCad schematic)
At the start: 5 parts, among them U1 DS18B20

Commit message: Kicadupdated
Parts:
- added R2, R3: 1K, Resistor_THT:R_Axial_DIN0207_L6.3mm_D2.5mm_P7.62mm_Horizontal, symbol Device:R
- added SOL+1, SOL-1: MountingHole_Pad, Connector_Pin:Pin_D1.0mm_L10.0mm, symbol Mechanical:MountingHole_Pad
Connections:
- net GND: now also R3.2, SOL-1.1
- net at A1.20 (A1): now also R2.1, R3.1
- new net: R2.2, SOL+1.1
Changed lines of the file:
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@@
   (junction (at 168.91 72.39) (diameter 0) (color 0 0 0 0)
   )
+  (junction (at 187.96 119.38) (diameter 0) (color 0 0 0 0)
+  )
+  (junction (at 165.1 107.95) (diameter 0) (color 0 0 0 0)
+  )
   (wire (pts (xy 168.91 86.36) (xy 168.91 72.39))
     (stroke (width 0) (type default))
@@
     (stroke (width 0) (type default))
   )
+  (wire (pts (xy 187.96 120.65) (xy 187.96 119.38))
+    (stroke (width 0) (type default))
+  )
+  (wire (pts (xy 148.59 77.47) (xy 165.1 77.47))
+    (stroke (width 0) (type default))
+  )
+  (wire (pts (xy 172.72 119.38) (xy 187.96 119.38))
+    (stroke (width 0) (type default))
+  )
+  (wire (pts (xy 165.1 77.47) (xy 165.1 107.95))
+    (stroke (width 0) (type default))
+  )
   (wire (pts (xy 148.59 74.93) (xy 176.53 74.93))
+    (stroke (width 0) (type default))
+  )
+  (wire (pts (xy 187.96 119.38) (xy 187.96 118.11))
+    (stroke (width 0) (type default))
+  )
+  (wire (pts (xy 165.1 107.95) (xy 165.1 119.38))
+    (stroke (width 0) (type default))
+  )
+  (wire (pts (xy 187.96 107.95) (xy 172.72 107.95))
     (stroke (width 0) (type default))
   )
@@
     )
   )
+  (symbol (lib_id "Device:R") (at 168.91 119.38 90) (unit 1)
+    (in_bom yes) (on_board yes) (dnp no) (fields_autoplaced)
+    (property "Reference" "R3" (at 168.91 113.03 90)
+      (effects (font (size 1.27 1.27)))
+    )
+    (property "Value" "1K" (at 168.91 115.57 90)
+      (effects (font (size 1.27 1.27)))
+    )
+    (property "Footprint" "Resistor_THT:R_Axial_DIN0207_L6.3mm_D2.5mm_P7.62mm_Horizontal" (at 168.91 121.158 90)
+      (effects (font (size 1.27 1.27)) hide)
+    )
+    (property "Datasheet" "~" (at 168.91 119.38 0)
+      (effects (font (size 1.27 1.27)) hide)
+    )
+    (pin "1")
+    (pin "2")
+    (instances
+      (project "ProjetSemestreKicad"
+        (path "/917d3087-48d5-488d-9cd0-e4f658acc78f"
+          (reference "R3") (unit 1)
+        )
+      )
+    )
+  )
+  (symbol (lib_id "Mechanical:MountingHole_Pad") (at 187.96 105.41 0) (unit 1)
+    (in_bom yes) (on_board yes) (dnp no) (fields_autoplaced)
+    (property "Reference" "SOL+1" (at 190.5 102.87 0)
+      (effects (font (size 1.27 1.27)) (justify left))
+    )
+    (property "Value" "MountingHole_Pad" (at 190.5 105.41 0)
+      (effects (font (size 1.27 1.27)) (justify left))
+    )
+    (property "Footprint" "Connector_Pin:Pin_D1.0mm_L10.0mm" (at 187.96 105.41 0)
+      (effects (font (size 1.27 1.27)) hide)
+    )
+    (property "Datasheet" "~" (at 187.96 105.41 0)
+      (effects (font (size 1.27 1.27)) hide)
+    )
+    (pin "1")
+    (instances
+      (project "ProjetSemestreKicad"
+        (path "/917d3087-48d5-488d-9cd0-e4f658acc78f"
+          (reference "SOL+1") (unit 1)
+        )
+      )
+    )
+  )
   (symbol (lib_id "power:GND") (at 135.89 100.33 0) (unit 1)
     (in_bom yes) (on_board yes) (dnp no) (fields_autoplaced)
@@
         (path "/917d3087-48d5-488d-9cd0-e4f658acc78f"
           (reference "#PWR02") (unit 1)
+        )
+      )
+    )
+  )
+  (symbol (lib_id "power:GND") (at 187.96 120.65 0) (unit 1)
+    (in_bom yes) (on_board yes) (dnp no) (fields_autoplaced)
+    (property "Reference" "#PWR05" (at 187.96 127 0)
+      (effects (font (size 1.27 1.27)) hide)
+    )
+    (property "Value" "GND" (at 187.96 125.73 0)
+      (effects (font (size 1.27 1.27)))
+    )
+    (property "Footprint" "" (at 187.96 120.65 0)
+      (effects (font (size 1.27 1.27)) hide)
+    )
+    (property "Datasheet" "" (at 187.96 120.65 0)
+      (effects (font (size 1.27 1.27)) hide)
+    )
+    (pin "1")
+    (instances
+      (project "ProjetSemestreKicad"
+        (path "/917d3087-48d5-488d-9cd0-e4f658acc78f"
+          (reference "#PWR05") (unit 1)
         )
       )
@@
     )
   )
+  (symbol (lib_id "Device:R") (at 168.91 107.95 90) (unit 1)
+    (in_bom yes) (on_board yes) (dnp no) (fields_autoplaced)
+    (property "Reference" "R2" (at 168.91 101.6 90)
+      (effects (font (size 1.27 1.27)))
+    )
+    (property "Value" "1K" (at 168.91 104.14 90)
+      (effects (font (size 1.27 1.27)))
+    )
+    (property "Footprint" "Resistor_THT:R_Axial_DIN0207_L6.3mm_D2.5mm_P7.62mm_Horizontal" (at 168.91 109.728 90)
+      (effects (font (size 1.27 1.27)) hide)
+    )
+    (property "Datasheet" "~" (at 168.91 107.95 0)
+      (effects (font (size 1.27 1.27)) hide)
+    )
+    (pin "1")
+    (pin "2")
+    (instances
+      (project "ProjetSemestreKicad"
+        (path "/917d3087-48d5-488d-9cd0-e4f658acc78f"
+          (reference "R2") (unit 1)
+        )
+      )
+    )
+  )
   (symbol (lib_id "power:GND") (at 105.41 49.53 0) (unit 1)
     (in_bom yes) (on_board yes) (dnp no) (fields_autoplaced)
@@
         )
       )
+    )
+  )
+  (symbol (lib_id "Mechanical:MountingHole_Pad") (at 187.96 115.57 0) (unit 1)
+    (in_bom yes) (on_board yes) (dnp no) (fields_autoplaced)
+    (property "Reference" "SOL-1" (at 190.5 113.03 0)
+      (effects (font (size 1.27 1.27)) (justify left))
+    )
+    (property "Value" "MountingHole_Pad" (at 190.5 115.57 0)
+      (effects (font (size 1.27 1.27)) (justify left))
+    )
+    (property "Footprint" "Connector_Pin:Pin_D1.0mm_L10.0mm" (at 187.96 115.57 0)
+      (effects (font (size 1.27 1.27)) hide)
+    )
+    (property "Datasheet" "~" (at 187.96 115.57 0)
+      (effects (font (size 1.27 1.27)) hide)
+    )
+    (pin "1")
+    (instances
+      (project "ProjetSemestreKicad"
+        (path "/917d3087-48d5-488d-9cd0-e4f658acc78f"
+          (reference "SOL-1") (unit 1)
+        )
+      )
