File: Hardware/Kicad/OptiprodV2/OptiprodV2.kicad_pcb (KiCad board)
At the start: 2 copper layers, 20 parts, among them U1 MCP6002-xMC, U2 BME280, U3 TL082, U4 TL082

Commit message: modified_kicad
Parts:
- added CS1: MountingHole_Pad, Connector_Pin:Pin_D1.0mm_L10.0mm, F.Cu at (144.8, 48.3)
- added GND1: MountingHole_Pad, Connector_Pin:Pin_D1.0mm_L10.0mm, F.Cu at (134.6, 48.2)
- added IN1: MountingHole_Pad, Connector_Pin:Pin_D1.0mm_L10.0mm, F.Cu at (101.6, 78.7)
- added SCL1: MountingHole_Pad, Connector_Pin:Pin_D1.0mm_L10.0mm, F.Cu at (137.2, 48.2)
- added SDA1: MountingHole_Pad, Connector_Pin:Pin_D1.0mm_L10.0mm, F.Cu at (139.7, 48.3)
- added SDO1: MountingHole_Pad, Connector_Pin:Pin_D1.0mm_L10.0mm, F.Cu at (142.2, 48.3)
- added VCC1: MountingHole_Pad, Connector_Pin:Pin_D1.0mm_L10.0mm, F.Cu at (132.1, 48.3)
- moved A2 2.54 mm to (94.0, 109.2)
Connections:
- A2 pad 3V3: unconnected-(A2-3.3V-Pad3V3) -> VCC
- U4 pad 4: (no net) -> GND
- U4 pad 8: (no net) -> Net-(U1C-V+)
Other:
- board text added: "BME680"

Commit message: modifiedkicad
Parts:
- removed 10K1, 12K1, 1K1, 1K2, 330R1, 330R2, 4.7K2, 470r1: R, Resistor_THT:R_Axial_DIN0204_L3.6mm_D1.6mm_P7.62mm_Horizontal
- removed D1, D2: D_Zener, Diode_THT:D_DO-35_SOD27_P7.62mm_Horizontal
- removed the D5 at (182.9, 83.8)
- removed U2: BME280, Package_LGA:Bosch_LGA-8_2.5x2.5mm_P0.65mm_ClockwisePinNumbering
- removed U3: TL082, Package_DIP:DIP-8_W7.62mm
- added DZ5: 1N4733, Diode_THT:D_A-405_P12.70mm_Horizontal, F.Cu at (111.8, 89.7)
- added DZ6: 1N4733, Diode_THT:D_A-405_P12.70mm_Horizontal, F.Cu at (111.8, 94.0)
- added Follower1: MountingHole_Pad, Connector_Pin:Pin_D1.0mm_L10.0mm, F.Cu at (116.8, 73.7)
- added Follower2: MountingHole_Pad, Connector_Pin:Pin_D1.0mm_L10.0mm, F.Cu at (116.8, 78.7)
- added R1: R, Resistor_THT:R_Axial_DIN0204_L3.6mm_D1.6mm_P7.62mm_Horizontal, F.Cu at (157.5, 95.7)
- added R2: R, Resistor_THT:R_Axial_DIN0204_L3.6mm_D1.6mm_P7.62mm_Horizontal, F.Cu at (167.6, 95.7)
- added R3: R, Resistor_THT:R_Axial_DIN0204_L3.6mm_D1.6mm_P7.62mm_Horizontal, F.Cu at (177.8, 88.1)
- added TRIM1: TrimPot_T73YEt_1k, PCM_Potentiometer_THT_US_AKL:Potentiometer_Bourns_3296W_Vertical, F.Cu at (152.4, 88.9)
- added TRIM2: TrimPot_T73YEt_1k, PCM_Potentiometer_THT_US_AKL:Potentiometer_Bourns_3296W_Vertical, F.Cu at (162.6, 88.9)
- added TRIM3: TrimPot_T73YEt_1k, PCM_Potentiometer_THT_US_AKL:Potentiometer_Bourns_3296W_Vertical, F.Cu at (172.7, 88.9)
- U1: value MCP6002-xMC -> DS18B20; footprint Package_DIP:DIP-8_W7.62mm -> Package_TO_SOT_THT:TO-92_Inline
- moved IN1 73.7 mm to (175.3, 78.7)
- moved 4.7K1 61.7 mm to (170.5, 71.8), turned to 90 degrees
- moved U1 56.2 mm to (175.3, 66.0), turned to -90 degrees
- moved U4 31.7 mm to (134.6, 96.5), turned to 90 degrees
- moved VCC1 30.6 mm to (129.6, 78.7), turned to 90 degrees
- moved GND1 28.4 mm to (129.5, 76.2), turned to 90 degrees
- moved SCL1 26.5 mm to (129.5, 73.7), turned to 90 degrees
- moved SDA1 25.0 mm to (129.6, 71.1), turned to 90 degrees
- moved SDO1 23.9 mm to (129.6, 68.6), turned to 90 degrees
- moved CS1 23.4 mm to (129.6, 66.0), turned to 90 degrees
Connections:
- 4.7K1 pad 1: Net-(U4A--) -> VCC
- 4.7K1 pad 2: Net-(U4B-+) -> Net-(U1-DQ)
- A2 pad 5V1: Net-(U1C-V+) -> VCC
- A2 pad A1: Net-(470r1-Pad2) -> unconnected-(A2-PadA1)
- A2 pad D20: unconnected-(A2-D20/SDA-PadD20) -> Net-(A2-D20/SDA)
- A2 pad D21: unconnected-(A2-D21/SCL-PadD21) -> Net-(A2-D21/SCL)
- SCL1 pad 1: unconnected-(SCL1-Pad1) -> Net-(A2-D21/SCL)
- SDA1 pad 1: unconnected-(SDA1-Pad1) -> Net-(A2-D20/SDA)
- U1 pad 1: Net-(470r1-Pad2) -> GND
- U1 pad 2: Net-(U1A--) -> Net-(U1-DQ)
- U1 pad 3: Net-(DZ3-K) -> VCC
- U4 pad 1: Net-(U4B-+) -> Net-(TRIM2-Right)
- U4 pad 2: Net-(U4A--) -> Net-(TRIM2-Center)
- U4 pad 5: Net-(U4B-+) -> Net-(TRIM2-Right)
- U4 pad 8: Net-(U1C-V+) -> VCC
Routing:
- net GND: track 0.00 -> 180.7 mm
- net VCC: track 0.00 -> 84.0 mm
- net Net-(DZ5-K): track 0.00 -> 75.8 mm
- net Net-(TRIM2-Right): track 0.00 -> 72.3 mm
- net Net-(D5-A): track 0.00 -> 68.6 mm
- net Net-(U4B--): track 0.00 -> 65.3 mm
- net Net-(D4-A): track 0.00 -> 63.7 mm
- net Net-(D3-A): track 0.00 -> 58.9 mm
- net Net-(A2-D21/SCL): track 0.00 -> 57.3 mm
- net Net-(A2-D20/SDA): track 0.00 -> 53.7 mm
- net Net-(TRIM2-Center): track 0.00 -> 49.9 mm
- net Net-(U3B-+): track 27.1 -> 0.00 mm
- net Net-(U1-DQ): track 0.00 -> 6.39 mm
- net Net-(DZ5-A): track 0.00 -> 4.25 mm
- net Net-(12K1-Pad2): track 1.32 -> 0.00 mm
- added copper zone on B.Cu, net GND
Other:
- board outline added: 101.6 x 53.3 mm

Commit message: PCBFinished?
Parts:
- removed D3, D4, D5: LED, LED_THT:LED_D3.0mm_Clear
- removed R1, R3: R, Resistor_THT:R_Axial_DIN0204_L3.6mm_D1.6mm_P7.62mm_Horizontal
- removed TRIM1, TRIM2, TRIM3: TrimPot_T73YEt_1k, PCM_Potentiometer_THT_US_AKL:Potentiometer_Bourns_3296W_Vertical
- added 1K1: TrimPot_T73YEt_1k, PCM_Potentiometer_THT_US_AKL:Potentiometer_Bourns_3296W_Vertical, F.Cu at (180.3, 101.6)
- added 1K2: R, Resistor_THT:R_Axial_DIN0204_L3.6mm_D1.6mm_P7.62mm_Horizontal, F.Cu at (123.2, 91.4)
- added G***: LOGO, Logo.preety:eurologo, B.Cu at (134.6, 81.3)
- added GNDS1: MountingHole_Pad, Connector_Pin:Pin_D1.0mm_L10.0mm, F.Cu at (175.3, 83.8)
- added SCL2: MountingHole_Pad, Connector_Pin:Pin_D1.0mm_L10.0mm, F.Cu at (175.3, 78.7)
- added SDA2: MountingHole_Pad, Connector_Pin:Pin_D1.0mm_L10.0mm, F.Cu at (175.3, 76.2)
- added VCCS1: MountingHole_Pad, Connector_Pin:Pin_D1.0mm_L10.0mm, F.Cu at (175.3, 81.4)
- moved VCC1 55.5 mm to (182.9, 63.5), turned to 180 degrees
- moved GND1 52.4 mm to (180.3, 63.5), turned to 180 degrees
- moved SCL1 49.3 mm to (177.8, 63.5), turned to 180 degrees
- moved 4.7K1 48.7 mm to (121.9, 74.9)
- moved SDA1 46.3 mm to (175.3, 63.5), turned to 180 degrees
- moved R2 44.5 mm to (123.2, 96.5), turned to 0 degrees
- moved SDO1 43.5 mm to (172.7, 63.5), turned to 180 degrees
- moved CS1 40.7 mm to (170.2, 63.5), turned to 180 degrees
- moved DZ6 27.7 mm to (110.0, 66.4), turned to -90 degrees
- moved TL082 25.4 mm to (109.2, 96.5)
- moved IN1 24.1 mm to (167.6, 101.6)
- moved DZ5 23.5 mm to (114.3, 66.4), turned to -90 degrees
- moved DS18B20 13.0 mm to (162.6, 63.5), turned to 0 degrees
- moved Follower1 10.2 mm to (116.8, 83.8)
- moved Follower2 5.68 mm to (119.4, 83.8)
- renumbered U1 to DS18B20, U4 to TL082
Connections:
- A2 pad 5V1: VCC -> VCCQ
- A2 pad D10: Net-(D3-A) -> unconnected-(A2-PadD10)
- A2 pad D11: Net-(D4-A) -> unconnected-(A2-PadD11)
- A2 pad D12: Net-(D5-A) -> unconnected-(A2-PadD12)
- A2 pad SCL: unconnected-(A2-PadSCL) -> Net-(A2-PadSCL)
- A2 pad SDA: unconnected-(A2-PadSDA) -> Net-(A2-PadSDA)
- TL082 pad 8: VCC -> VCCQ
Routing:
- net GND: track 180.7 -> 0.00 mm
- net VCCQ: track 0.00 -> 87.8 mm
- net Net-(A2-PadSCL): track 0.00 -> 71.1 mm
- net Net-(A2-PadSDA): track 0.00 -> 70.9 mm
- net Net-(D5-A): track 68.6 -> 0.00 mm
- net Net-(D4-A): track 63.7 -> 0.00 mm
- net Net-(D3-A): track 58.9 -> 0.00 mm
- net Net-(A2-D21/SCL): track 57.3 -> 6.13 mm
- net Net-(1K1-Right): track 0.00 -> 48.7 mm
- net Net-(A2-D20/SDA): track 53.7 -> 6.10 mm
- net Net-(TL082B-+): track 72.3 -> 34.0 mm
- net Net-(DS18B20-DQ): track 6.39 -> 44.1 mm
- net VCC: track 84.0 -> 109.6 mm
- net Net-(1K1-Center): track 49.9 -> 70.1 mm
- net Net-(TL082B--): track 65.3 -> 46.5 mm
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Other:
- board text added: "MoneyMoni Made By Meriam Melvyn Felipe Haoyu Zhuodong EPF2023"
- board text added: "SCREEN"

Commit message: pcbfinished?
Parts:
- added G***: LOGO, Logo.preety:ElfamosoMelvyn5mm, B.Cu at (116.8, 104.1)
- moved G*** 5.08 mm to (129.5, 81.3)

Commit message: PCBFinishedforreal??
Parts:
- added G***: LOGO, Logo.preety:FelipeBarbaste, B.Cu at (114.3, 101.6)
- added G***: LOGO, Logo.preety:ZhuodongKangAutoportrait, B.Cu at (109.2, 101.6)
- moved G*** 5.68 mm to (121.9, 101.6)

Commit message: stencilcreated
Parts:
- added G***: LOGO, Logo.preety:Moneymoney30, F.Cu at (142.2, 81.3)
- added G***: LOGO, Logo.preety:EPFLOGO15MM, B.Cu at (180.3, 88.9)
- added G***hjgugctyv: LOGO, Logo.preety:Moneymoney25, B.Cu at (142.2, 66.0)
- added GNDIN1: MountingHole_Pad, Connector_Pin:Pin_D1.0mm_L10.0mm, F.Cu at (170.2, 99.1)
- moved IN1 2.54 mm to (170.2, 101.6)
- moved 1K1 1.52 mm to (181.9, 101.6)
- moved 1K2 1.52 mm to (124.7, 91.4)
- moved 4.7K1 1.52 mm to (123.4, 74.9)
- moved 51K1 1.52 mm to (124.7, 96.5)
- moved A2 1.52 mm to (95.5, 109.2)
- moved CS1 1.52 mm to (171.7, 63.5)
- moved DS18B20 1.52 mm to (164.1, 63.5)
- moved DZ5 1.52 mm to (115.8, 66.4)
- moved DZ6 1.52 mm to (111.6, 66.4)
- moved Follower1 1.52 mm to (118.4, 83.8)
- moved Follower2 1.52 mm to (120.9, 83.8)
- moved G***LK 1.52 mm to (123.4, 101.6)
- moved G***fdwsw 1.52 mm to (131.1, 81.3)
- moved G***jgj 1.52 mm to (115.8, 101.6)
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- renumbered R2 to 51K1, G*** to G***LK, G*** to G***fdwsw, G*** to G***jgj, G*** to G***lkkjb, TL082 to MCP602
Routing:
- net VCC: track 109.6 -> 121.2 mm
- net VCCQ: track 87.8 -> 86.3 mm
- net Net-(A2-PadSDA): track 70.9 -> 69.5 mm
- net Net-(DZ5-K): track 91.1 -> 92.1 mm
- net Net-(A2-PadSCL): track 71.1 -> 72.0 mm
- net Net-(MCP602B-+): track 34.0 -> 34.6 mm
Other:
- board size 101.6 x 53.3 mm -> 88.9 x 53.3 mm

Commit message: PCBlastCommit?
Parts:
- removed G***jgj: LOGO, Logo.preety:FelipeBarbaste
- removed G***lkkjb: LOGO, Logo.preety:ZhuodongKangAutoportrait
- added G!kxxgjh: LOGO, Logo.preety:EPFLOGO15MM, F.Cu at (180.3, 91.4)
- added G:jgggjfuy: LOGO, Logo.preety:ZHK8MM, F.Cu at (137.2, 101.6)
- added G:jgggjfuy: LOGO, Logo.preety:ZHK8MM, B.Cu at (137.2, 101.6)
- added G;;vhfc: LOGO, Logo.preety:15mmlogoRW.kicadnonreverse_mod, F.Cu at (147.3, 101.6)
- added G;;vhfc: LOGO, Logo.preety:15mmlogoRW.kicadnonreverse_mod, B.Cu at (147.3, 101.6)
- added Gjchfmljkgjhv: LOGO, Logo.preety:Haoyu8MM, F.Cu at (129.5, 101.6)
- added Gjchfmljkgjhv: LOGO, Logo.preety:Haoyu8MM, B.Cu at (129.5, 101.6)
- added Gkvghgcfc: MountingHole_Pad, Connector_Pin:Pin_D1.0mm_L10.0mm, F.Cu at (170.2, 96.5)
- added hfihgxgfx: LOGO, Logo.preety:FelipeBarbaste10mm, F.Cu at (121.9, 101.6)
- added hfihgxgfx: LOGO, Logo.preety:FelipeBarbaste10mm, B.Cu at (119.4, 101.6)
- G***LK: moved to F.Cu
- moved G***LK 12.6 mm to (114.5, 92.7), turned to 90 degrees
- moved G!kxxgjh 2.54 mm to (180.3, 91.4)
- renumbered G*** to G!kxxgjh
Routing:
- net Net-(1K1-Center): track 70.1 -> 73.2 mm
- net Net-(1K1-Right): track 48.7 -> 49.3 mm
