File: Hardware/Kicad/OptiprodV2/OptiprodV2.kicad_sch (KiCad schematic)
At the start: 17 parts, among them U1 MCP6002-xMC, U2 BME280, U3 TL082

Commit message: commit2.2.1
Parts:
- renumbered 330R to 330R1, 4.7K to 4.7K1
Changed lines of the file:
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@@
   (symbol (lib_id "Device:R") (at 41.91 54.61 0) (unit 1)
     (in_bom yes) (on_board yes) (dnp no) (fields_autoplaced)
-    (property "Reference" "330R" (at 44.45 53.34 0)
+    (property "Reference" "330R1" (at 44.45 53.34 0)
       (effects (font (size 1.27 1.27)) (justify left))
     )
@@
       (project "OptiprodV2"
         (path "/19de4d2e-807d-4105-96d5-33b255df2ff3"
-          (reference "330R") (unit 1)
+          (reference "330R1") (unit 1)
         )
       )
@@
   (symbol (lib_id "Device:R") (at 54.61 49.53 90) (unit 1)
     (in_bom yes) (on_board yes) (dnp no) (fields_autoplaced)
-    (property "Reference" "4.7K" (at 54.61 43.18 90)
+    (property "Reference" "4.7K1" (at 54.61 43.18 90)
       (effects (font (size 1.27 1.27)))
     )
@@
       (project "OptiprodV2"
         (path "/19de4d2e-807d-4105-96d5-33b255df2ff3"
-          (reference "4.7K") (unit 1)
+          (reference "4.7K1") (unit 1)
         )
       )
