File: Hardware/Kicad/OptiprodV2/OptiprodV2.kicad_sch (KiCad schematic)
At the start: 30 parts, among them U1 MCP6002-xMC, U2 BME680, U3 TL082, U4 TL082

Commit message: updatekicad
Parts:
- removed U2: BME680, symbol Sensor:BME680
- added unit 3 of U4
Connections:
- net GND: now also U4.4 (V-)
- net at A2.5V1 (5V), U1.8 (V+), U3.8 (V+): now also U4.8 (V+)
Other:
- moved on the sheet: CS1, SDA1

Commit message: moded
Connections:
- net at SDA1.1: now also A2.D20 (D20/SDA)
- net at SCL1.1: now also A2.D21 (D21/SCL)
Other:
- moved on the sheet: CS1, GND1, SCL1, SDA1, SDO1, VCC1

Commit message: modifiedkicad
Parts:
- removed 12K1, 1K1, 1K2, 330R2, 4.7K2, 470r1: R, Resistor_THT:R_Axial_DIN0204_L3.6mm_D1.6mm_P7.62mm_Horizontal, symbol Device:R
- removed DZ1, DZ2, DZ3, DZ4: 1N4733, Diode_THT_AKL:D_DO-41_SOD81_P7.62mm_Horizontal_Zener, symbol PCM_Diode_Zener_AKL:1N4733
- removed U1: MCP6002-xMC, Package_DIP:DIP-8_W7.62mm, symbol Amplifier_Operational:MCP6002-xMC
- removed U3: TL082, Package_DIP:DIP-8_W7.62mm, symbol Amplifier_Operational:TL082
- added 4.7K1: R, Resistor_THT:R_Axial_DIN0204_L3.6mm_D1.6mm_P7.62mm_Horizontal, symbol Device:R
- added Follower1, Follower2: MountingHole_Pad, Connector_Pin:Pin_D1.0mm_L10.0mm, symbol Mechanical:MountingHole_Pad
- added TRIM1, TRIM2, TRIM3: TrimPot_T73YEt_1k, PCM_Potentiometer_THT_US_AKL:Potentiometer_Bourns_3296W_Vertical, symbol PCM_4ms_Potentiometer:TrimPot_T73YEt_1k
- added U1: DS18B20, Package_TO_SOT_THT:TO-92_Inline, symbol Sensor_Temperature:DS18B20
- DZ5, DZ6: footprint Diode_THT_AKL:D_DO-41_SOD81_P7.62mm_Horizontal_Zener -> Diode_THT:D_A-405_P12.70mm_Horizontal
- renumbered 10K1 to R1, 4.7K1 to R2, 330R1 to R3
Connections:
- net GND: now also TRIM1.2 (Center), TRIM3.3 (Right), U1.1 (GND)
- net VCC: now also A2.5V1 (5V), U4.8 (V+), 4.7K1.1, U1.3 (V_{DD})
- net at DZ5.1 (K), IN1.1, R1.1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: now also TRIM1.3 (Right)
- net at A2.A0, U4.6 (-), U4.7: now also Follower1.1
- net at R2.2, U4.1, U4.5 (+): now also Follower2.1, TRIM2.3 (Right)
- net at R2.1, R3.1, U4.2 (-): now also TRIM2.2 (Center), TRIM3.2 (Center)
- new net: 4.7K1.2, U1.2 (DQ)
Other:
- moved on the sheet: DZ5, DZ6, IN1, R1, R2, R3, U4A, U4B, U4C

Commit message: PCBFinished?
Parts:
- removed D3, D4, D5: LED, LED_THT:LED_D3.0mm_Clear, symbol Device:LED
- removed R1, R3: R, Resistor_THT:R_Axial_DIN0204_L3.6mm_D1.6mm_P7.62mm_Horizontal, symbol Device:R
- removed TRIM1, TRIM2: TrimPot_T73YEt_1k, PCM_Potentiometer_THT_US_AKL:Potentiometer_Bourns_3296W_Vertical, symbol PCM_4ms_Potentiometer:TrimPot_T73YEt_1k
- added 1K2: R, Resistor_THT:R_Axial_DIN0204_L3.6mm_D1.6mm_P7.62mm_Horizontal, symbol Device:R
- added GNDS1, SCL2, SDA2, VCCS1: MountingHole_Pad, Connector_Pin:Pin_D1.0mm_L10.0mm, symbol Mechanical:MountingHole_Pad
- renumbered TRIM3 to 1K1, U1 to DS18B20, U4 to TL082
Connections:
- net GND: now also 1K2.1, GNDS1.1; no longer 1K1.3 (Right)
- net VCC: no longer A2.5V1 (5V), TL082.8 (V+)
- net at A2.SCL: now also SCL2.1
- net at A2.SDA: now also SDA2.1
- new net: 1K1.3 (Right), 1K2.2
- new net VCCQ: A2.5V1 (5V), TL082.8 (V+), VCCS1.1
Other:
- moved on the sheet: SCL1

Commit message: PCBFinishedforreal??
Parts:
- renumbered R2 to 51K
Changed lines of the file:
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@@
   (symbol (lib_id "Device:R") (at 76.2 105.41 90) (unit 1)
     (in_bom yes) (on_board yes) (dnp no) (fields_autoplaced)
-    (property "Reference" "R2" (at 76.2 99.06 90)
+    (property "Reference" "51K" (at 76.2 99.06 90)
       (effects (font (size 1.27 1.27)))
     )
@@
       (project "OptiprodV2"
         (path "/19de4d2e-807d-4105-96d5-33b255df2ff3"
-          (reference "R2") (unit 1)
+          (reference "51K") (unit 1)
         )
       )

Commit message: PCBlastCommit?
Parts:
- added GNDIN1: MountingHole_Pad, Connector_Pin:Pin_D1.0mm_L10.0mm, symbol Mechanical:MountingHole_Pad
- renumbered 51K to 51K1, TL082 to MCP602
Connections:
- net GND: now also GNDIN1.1
Changed lines of the file:
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@@
   (symbol (lib_id "Amplifier_Operational:TL082") (at 116.84 157.48 270) (unit 3)
     (in_bom yes) (on_board yes) (dnp no) (fields_autoplaced)
-    (property "Reference" "TL082" (at 116.84 149.86 90)
+    (property "Reference" "MCP602" (at 116.84 149.86 90)
       (effects (font (size 1.27 1.27)))
     )
@@
       (project "OptiprodV2"
         (path "/19de4d2e-807d-4105-96d5-33b255df2ff3"
-          (reference "TL082") (unit 3)
+          (reference "MCP602") (unit 3)
         )
       )
@@
         (path "/19de4d2e-807d-4105-96d5-33b255df2ff3"
           (reference "IN1") (unit 1)
+        )
+      )
+    )
+  )
+  (symbol (lib_id "Mechanical:MountingHole_Pad") (at 54.61 54.61 0) (unit 1)
+    (in_bom yes) (on_board yes) (dnp no) (fields_autoplaced)
+    (property "Reference" "GNDIN1" (at 57.15 52.07 0)
+      (effects (font (size 1.27 1.27)) (justify left))
+    )
+    (property "Value" "MountingHole_Pad" (at 57.15 54.61 0)
+      (effects (font (size 1.27 1.27)) (justify left))
+    )
+    (property "Footprint" "Connector_Pin:Pin_D1.0mm_L10.0mm" (at 54.61 54.61 0)
+      (effects (font (size 1.27 1.27)) hide)
+    )
+    (property "Datasheet" "~" (at 54.61 54.61 0)
+      (effects (font (size 1.27 1.27)) hide)
+    )
+    (pin "1")
+    (instances
+      (project "OptiprodV2"
+        (path "/19de4d2e-807d-4105-96d5-33b255df2ff3"
+          (reference "GNDIN1") (unit 1)
         )
       )
@@
   (symbol (lib_id "Amplifier_Operational:TL082") (at 71.12 96.52 0) (unit 1)
     (in_bom yes) (on_board yes) (dnp no) (fields_autoplaced)
-    (property "Reference" "TL082" (at 71.12 86.36 0)
+    (property "Reference" "MCP602" (at 71.12 86.36 0)
       (effects (font (size 1.27 1.27)))
     )
@@
       (project "OptiprodV2"
         (path "/19de4d2e-807d-4105-96d5-33b255df2ff3"
-          (reference "TL082") (unit 1)
+          (reference "MCP602") (unit 1)
         )
       )
@@
   (symbol (lib_id "Amplifier_Operational:TL082") (at 102.87 99.06 0) (unit 2)
     (in_bom yes) (on_board yes) (dnp no) (fields_autoplaced)
-    (property "Reference" "TL082" (at 102.87 88.9 0)
+    (property "Reference" "MCP602" (at 102.87 88.9 0)
       (effects (font (size 1.27 1.27)))
     )
@@
       (project "OptiprodV2"
         (path "/19de4d2e-807d-4105-96d5-33b255df2ff3"
-          (reference "TL082") (unit 2)
+          (reference "MCP602") (unit 2)
         )
       )
@@
   (symbol (lib_id "Device:R") (at 76.2 105.41 90) (unit 1)
     (in_bom yes) (on_board yes) (dnp no) (fields_autoplaced)
-    (property "Reference" "51K" (at 76.2 99.06 90)
+    (property "Reference" "51K1" (at 76.2 99.06 90)
       (effects (font (size 1.27 1.27)))
     )
@@
       (project "OptiprodV2"
         (path "/19de4d2e-807d-4105-96d5-33b255df2ff3"
-          (reference "51K") (unit 1)
-        )
-      )
+          (reference "51K1") (unit 1)
+        )
+      )
+    )
+  )
+  (symbol (lib_id "PCM_4ms_Power-symbol:GND") (at 54.61 57.15 0) (unit 1)
+    (in_bom yes) (on_board yes) (dnp no) (fields_autoplaced)
+    (property "Reference" "#PWR05" (at 54.61 63.5 0)
+      (effects (font (size 1.27 1.27)) hide)
+    )
+    (property "Value" "GND" (at 54.61 62.23 0)
+      (effects (font (size 1.27 1.27)))
+    )
+    (property "Footprint" "" (at 54.61 57.15 0)
+      (effects (font (size 1.27 1.27)) hide)
+    )
+    (property "Datasheet" "" (at 54.61 57.15 0)
+      (effects (font (size 1.27 1.27)) hide)
+    )
+    (pin "1")
+    (instances
+      (project "OptiprodV2"
+        (path "/19de4d2e-807d-4105-96d5-33b255df2ff3"
+          (reference "#PWR05") (unit 1)
+        )
+      )
