File: Hardware/Kicad/OptiprodV2/_autosave-OptiprodV2.kicad_pcb (KiCad board)
At the start: 2 copper layers, 27 parts, among them U1 MCP6002-xMC, U2 BME280, U3 TL082, U4 TL082

Commit message: modified_kicad
Parts:
- removed the D5 at (182.9, 83.8)
- moved SDA1 46.8 mm to (172.8, 81.4)
- moved CS1 46.8 mm to (177.8, 81.4)
- moved GND1 46.8 mm to (167.7, 81.4)
- moved SCL1 46.8 mm to (170.2, 81.4)
- moved SDO1 46.8 mm to (175.3, 81.4)
- moved VCC1 46.8 mm to (165.1, 81.4)
Routing:
- net GND: track 0.00 -> 181.2 mm
- net Net-(U1C-V+): track 0.00 -> 77.5 mm
- net Net-(D5-A): track 0.00 -> 68.6 mm
- net Net-(D4-A): track 0.00 -> 63.7 mm
- net Net-(U3B--): track 0.00 -> 59.9 mm
- net Net-(D3-A): track 0.00 -> 58.9 mm
- net Net-(470r1-Pad2): track 0.00 -> 55.6 mm
- net VCC: track 0.00 -> 48.2 mm
- net Net-(U1A--): track 0.00 -> 31.6 mm
- net Net-(U4A--): track 0.00 -> 31.1 mm
- net Net-(U4B-+): track 0.00 -> 30.8 mm
- net Net-(U3A--): track 0.00 -> 30.0 mm
- net Net-(DZ5-K): track 0.00 -> 27.3 mm
- net Net-(12K1-Pad2): track 1.32 -> 12.7 mm
- net Net-(1K2-Pad2): track 0.00 -> 8.92 mm
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- added copper zone on B.Cu, net GND
Other:
- board outline added: 101.6 x 53.3 mm
