File: Hardware/Kicad/OptiprodV2/_autosave-OptiprodV2.kicad_sch (KiCad schematic)
At the start: 22 parts

Commit message: codesformeriam
Parts:
- renumbered TL82 to MCP602
Changed lines of the file:
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@@
   (symbol (lib_id "Amplifier_Operational:TL082") (at 116.84 157.48 270) (unit 3)
     (in_bom yes) (on_board yes) (dnp no) (fields_autoplaced)
-    (property "Reference" "TL82" (at 116.84 149.86 90)
+    (property "Reference" "MCP602" (at 116.84 149.86 90)
       (effects (font (size 1.27 1.27)))
     )
@@
       (project "OptiprodV2"
         (path "/19de4d2e-807d-4105-96d5-33b255df2ff3"
-          (reference "TL82") (unit 3)
+          (reference "MCP602") (unit 3)
         )
       )
@@
   (symbol (lib_id "Amplifier_Operational:TL082") (at 71.12 96.52 0) (unit 1)
     (in_bom yes) (on_board yes) (dnp no) (fields_autoplaced)
-    (property "Reference" "TL82" (at 71.12 86.36 0)
+    (property "Reference" "MCP602" (at 71.12 86.36 0)
       (effects (font (size 1.27 1.27)))
     )
@@
       (project "OptiprodV2"
         (path "/19de4d2e-807d-4105-96d5-33b255df2ff3"
-          (reference "TL82") (unit 1)
+          (reference "MCP602") (unit 1)
         )
       )
@@
   (symbol (lib_id "Amplifier_Operational:TL082") (at 102.87 99.06 0) (unit 2)
     (in_bom yes) (on_board yes) (dnp no) (fields_autoplaced)
-    (property "Reference" "TL82" (at 102.87 88.9 0)
+    (property "Reference" "MCP602" (at 102.87 88.9 0)
       (effects (font (size 1.27 1.27)))
     )
@@
       (project "OptiprodV2"
         (path "/19de4d2e-807d-4105-96d5-33b255df2ff3"
-          (reference "TL82") (unit 2)
-        )
-      )
+          (reference "MCP602") (unit 2)
+        )
+      )

Commit message: stencilcreated
Parts:
- added GNDIN1: MountingHole_Pad, Connector_Pin:Pin_D1.0mm_L10.0mm, symbol Mechanical:MountingHole_Pad
Connections:
- net GND: now also GNDIN1.1
Changed lines of the file:
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@@
+    )
+  )
+  (symbol (lib_id "Mechanical:MountingHole_Pad") (at 54.61 54.61 0) (unit 1)
+    (in_bom yes) (on_board yes) (dnp no) (fields_autoplaced)
+    (property "Reference" "GNDIN1" (at 57.15 52.07 0)
+      (effects (font (size 1.27 1.27)) (justify left))
+    )
+    (property "Value" "MountingHole_Pad" (at 57.15 54.61 0)
+      (effects (font (size 1.27 1.27)) (justify left))
+    )
+    (property "Footprint" "Connector_Pin:Pin_D1.0mm_L10.0mm" (at 54.61 54.61 0)
+      (effects (font (size 1.27 1.27)) hide)
+    )
+    (property "Datasheet" "~" (at 54.61 54.61 0)
+      (effects (font (size 1.27 1.27)) hide)
+    )
+    (pin "1")
+    (instances
+      (project "OptiprodV2"
+        (path "/19de4d2e-807d-4105-96d5-33b255df2ff3"
+          (reference "GNDIN1") (unit 1)
+        )
+      )
     )
   )
@@
         )
       )
+    )
+  )
+  (symbol (lib_id "PCM_4ms_Power-symbol:GND") (at 54.61 57.15 0) (unit 1)
+    (in_bom yes) (on_board yes) (dnp no) (fields_autoplaced)
+    (property "Reference" "#PWR05" (at 54.61 63.5 0)
+      (effects (font (size 1.27 1.27)) hide)
+    )
+    (property "Value" "GND" (at 54.61 62.23 0)
+      (effects (font (size 1.27 1.27)))
+    )
+    (property "Footprint" "" (at 54.61 57.15 0)
+      (effects (font (size 1.27 1.27)) hide)
+    )
+    (property "Datasheet" "" (at 54.61 57.15 0)
+      (effects (font (size 1.27 1.27)) hide)
+    )
+    (pin "1")
+    (instances
+      (project "OptiprodV2"
+        (path "/19de4d2e-807d-4105-96d5-33b255df2ff3"
+          (reference "#PWR05") (unit 1)
+        )
+      )
