File: Hardware/Kicad/OptiprodCommand/OptiprodV2.kicad_pcb (KiCad board)
At the start: 2 copper layers, 88.9 x 53.3 mm, 38 parts

Commit message: correctedKicad
Parts:
- removed the GNDIN1 at (170.2, 99.1)
- added GNDIN2: MountingHole_Pad, Connector_Pin:Pin_D1.0mm_L10.0mm, F.Cu at (170.2, 101.6)
- DS18B20: footprint Package_TO_SOT_THT:TO-92_Inline -> Package_TO_SOT_THT:TO-92_Inline_Wide
- I IUG UYGHIUNIJ?CU NC4R3H44IRB: renamed from hfihgxgfx
- KJHHIB9UYG 8TBYFI TG8Y : renamed from G!kxxgjh
- eopjohkbihvçh,&iàéahihazdnçià?ADZO0IERZGDSQHJ32GN0JCH3 0KCINR39XNGZHENCHZUNVYHIUNHC2NIUN3: renamed from G***
- pjbiçh u_tftf: renamed from hfihgxgfx
- moved 4.7K1 35.9 mm to (157.5, 63.5), turned to 180 degrees
- moved IN1 2.54 mm to (170.2, 99.1)
- moved GNDS1 2.50 mm to (176.8, 86.3)
- moved SCL2 2.50 mm to (176.8, 81.2)
- moved VCCS1 2.50 mm to (176.8, 83.9)
- moved SDA2 2.50 mm to (176.8, 78.7)
- moved DS18B20 1.52 mm to (162.6, 63.5)
- renumbered G:jgggjfuy to G:jgggjfuykjfèdtrdètuvf_yvc, Gkvghgcfc to GNDIN1, G***hjgugctyv to Ghhhgfcccdcdfcfgvfvfvdfcxdrdsqaqhjgugctyv, G!kxxgjh to azertyuxcvbngfdsqzert, Gjchfmljkgjhv to ggfrtdrdpopop, G***fdwsw to hhfttyhgfdssaazzqwxcvbn,kpo, G;;vhfc to khojhvgvgvjhbhjvuuuzuaanhhsrrsnnf1456789876432112345678765432123467U8765432123456765432134567UI, G;;vhfc to uhuhh
Connections:
- A2 pad A1: unconnected-(A2-PadA1) -> Net-(DS18B20-DQ)
Routing:
- net VCC: track 121.2 -> 96.5 mm
- net Net-(DS18B20-DQ): track 44.1 -> 59.8 mm
- net Net-(1K1-Center): track 73.2 -> 71.3 mm
- net Net-(A2-PadSDA): track 69.5 -> 68.6 mm
- net VCCQ: track 86.3 -> 87.2 mm
- net Net-(MCP602B-+): track 34.6 -> 34.1 mm
Other:
- board text added: "Follower"
