File: Hardware/Kicad/OptiprodCommand/OptiprodV2.kicad_sch (KiCad schematic)
At the start: 23 parts

Commit message: kicad_update
Connections:
- net at A2.A1: now also 4.7K1.2, DS18B20.2 (DQ)
Changed lines of the file:
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@@
   (junction (at 80.01 96.52) (diameter 0) (color 0 0 0 0)
+  )
+  (junction (at 66.04 148.59) (diameter 0) (color 0 0 0 0)
   )
   (junction (at 142.24 172.72) (diameter 0) (color 0 0 0 0)
@@
     (stroke (width 0) (type default))
   )
+  (wire (pts (xy 66.04 148.59) (xy 66.04 152.4))
+    (stroke (width 0) (type default))
+  )
   (wire (pts (xy 38.1 93.98) (xy 63.5 93.98))
+    (stroke (width 0) (type default))
+  )
+  (wire (pts (xy 134.62 101.6) (xy 134.62 148.59))
     (stroke (width 0) (type default))
   )
@@
     (stroke (width 0) (type default))
   )
-  (wire (pts (xy 66.04 144.78) (xy 66.04 152.4))
+  (wire (pts (xy 66.04 144.78) (xy 66.04 148.59))
     (stroke (width 0) (type default))
   )
@@
     (stroke (width 0) (type default))
   )
+  (wire (pts (xy 142.24 101.6) (xy 134.62 101.6))
+    (stroke (width 0) (type default))
+  )
   (wire (pts (xy 63.5 105.41) (xy 63.5 99.06))
     (stroke (width 0) (type default))
@@
     (stroke (width 0) (type default))
   )
+  (wire (pts (xy 134.62 148.59) (xy 66.04 148.59))
+    (stroke (width 0) (type default))
+  )

Commit message: correctedKicad
Parts:
- added GNDIN2: MountingHole_Pad, Connector_Pin:Pin_D1.0mm_L10.0mm, symbol Mechanical:MountingHole_Pad
- DS18B20: footprint Package_TO_SOT_THT:TO-92_Inline -> Package_TO_SOT_THT:TO-92_Inline_Wide
Connections:
- net GND: now also GNDIN2.1
Changed lines of the file:
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@@
       (effects (font (size 1.27 1.27)) (justify right))
     )
-    (property "Footprint" "Package_TO_SOT_THT:TO-92_Inline" (at 33.02 158.75 0)
+    (property "Footprint" "Package_TO_SOT_THT:TO-92_Inline_Wide" (at 33.02 158.75 0)
       (effects (font (size 1.27 1.27)) hide)
     )
@@
         (path "/19de4d2e-807d-4105-96d5-33b255df2ff3"
           (reference "#PWR07") (unit 1)
+        )
+      )
+    )
+  )
+  (symbol (lib_id "PCM_4ms_Power-symbol:GND") (at 34.29 68.58 0) (unit 1)
+    (in_bom yes) (on_board yes) (dnp no) (fields_autoplaced)
+    (property "Reference" "#PWR011" (at 34.29 74.93 0)
+      (effects (font (size 1.27 1.27)) hide)
+    )
+    (property "Value" "GND" (at 34.29 73.66 0)
+      (effects (font (size 1.27 1.27)))
+    )
+    (property "Footprint" "" (at 34.29 68.58 0)
+      (effects (font (size 1.27 1.27)) hide)
+    )
+    (property "Datasheet" "" (at 34.29 68.58 0)
+      (effects (font (size 1.27 1.27)) hide)
+    )
+    (pin "1")
+    (instances
+      (project "OptiprodV2"
+        (path "/19de4d2e-807d-4105-96d5-33b255df2ff3"
+          (reference "#PWR011") (unit 1)
         )
       )
@@
         )
       )
+    )
+  )
+  (symbol (lib_id "Mechanical:MountingHole_Pad") (at 34.29 66.04 0) (unit 1)
+    (in_bom yes) (on_board yes) (dnp no) (fields_autoplaced)
+    (property "Reference" "GNDIN2" (at 36.83 63.5 0)
+      (effects (font (size 1.27 1.27)) (justify left))
+    )
+    (property "Value" "MountingHole_Pad" (at 36.83 66.04 0)
+      (effects (font (size 1.27 1.27)) (justify left))
+    )
+    (property "Footprint" "Connector_Pin:Pin_D1.0mm_L10.0mm" (at 34.29 66.04 0)
+      (effects (font (size 1.27 1.27)) hide)
+    )
+    (property "Datasheet" "~" (at 34.29 66.04 0)
+      (effects (font (size 1.27 1.27)) hide)
+    )
+    (pin "1")
+    (instances
+      (project "OptiprodV2"
+        (path "/19de4d2e-807d-4105-96d5-33b255df2ff3"
+          (reference "GNDIN2") (unit 1)
+        )
+      )
