File: Hardware/Kicad/OptiprodProduct/OptiprodV2.kicad_sch (KiCad schematic)
At the start: 26 parts

Commit message: readyforproduction!!!!!!
Connections:
- net VCCQ: now also A2.5V3 (5V), A2.5V4 (5V)
Changed lines of the file:
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@@
   (junction (at 63.5 105.41) (diameter 0) (color 0 0 0 0)
+  )
+  (junction (at 142.24 154.94) (diameter 0) (color 0 0 0 0)
   )
   (junction (at 142.24 170.18) (diameter 0) (color 0 0 0 0)
@@
   )
   (junction (at 76.2 148.59) (diameter 0) (color 0 0 0 0)
+  )
+  (junction (at 142.24 157.48) (diameter 0) (color 0 0 0 0)
   )
   (junction (at 58.42 142.24) (diameter 0) (color 0 0 0 0)
@@
     (stroke (width 0) (type default))
   )
+  (wire (pts (xy 142.24 154.94) (xy 142.24 157.48))
+    (stroke (width 0) (type default))
+  )
   (wire (pts (xy 142.24 99.06) (xy 110.49 99.06))
     (stroke (width 0) (type default))
@@
     (stroke (width 0) (type default))
   )
+  (wire (pts (xy 142.24 157.48) (xy 142.24 160.02))
+    (stroke (width 0) (type default))
+  )
